File: pcb/3WayESP32/3WayESP32.kicad_sch (KiCad schematic)
At the start: 8 parts, among them J1 Conn_01x06_Pin, J2 Conn_01x06_Pin, J3 Conn_01x06_Pin

Commit message: Plated mounting holes
Parts:
- removed H1, H2, H3, H4: MountingHole, MountingHole:MountingHole_3.2mm_M3, symbol Mechanical:MountingHole
- added H1, H2: MountingHole_Pad, MountingHole:MountingHole_3.2mm_M3_DIN965_Pad, symbol Mechanical:MountingHole_Pad
- added H3, H4: MountingHole_Pad, MountingHole:MountingHole_3.2mm_M3_Pad, symbol Mechanical:MountingHole_Pad
Connections:
- net GND: now also H1.1, H2.1, H3.1, H4.1
- no-connect marks 0 -> 8
